File: PCB/robo-con-Wi-Fi-v2/robo-con-Wi-Fi-v2.kicad_pcb (KiCad board)
At the start: 4 copper layers, 86 x 62 mm, 107 parts, among them J1 Conn_01x04, J10 Conn_01x06, J2 SMA-J, J4 Conn_01x01, J5 Conn_01x02, J6 Conn_01x01, J7 Conn_01x06, J8 Conn_01x01, J9 Conn_01x01, SW1 SW_Push, SW3 SW_Push, SW4 SW_Push, SW5 SW_Push_SPDT, SW6 SW_Push_SPDT, SW7 SW_Push_SPDT, U10 MCP73831-2-OT, U11 LM66100DCK, U15 LM66100DCK, U18 USB_Type-C, U2 LBEE5HY2FY, U3 FT234XD, U4 MCP1727-1802xMF, U5 RKJXV122400R, U6 LD39200PU33R, U7 RKJXV122400R, U8 STM32H7A3RGTx, Y2 XRCGB25M000FFS1AR0

Commit message: update PCB
Parts:
- removed J10, J7: Conn_01x06, Connector_JST:JST_ZH_B6B-ZR_1x06_P1.50mm_Vertical
- added J11: Conn_01x05, Connector_JST:JST_ZH_B5B-ZR_1x05_P1.50mm_Vertical, F.Cu at (205.3, 65.9)
- added J3: Conn_01x05, Connector_JST:JST_ZH_B5B-ZR_1x05_P1.50mm_Vertical, F.Cu at (134.7, 59.1)
- J8, J9: moved to B.Cu
- moved J4 134.3 mm to (210.3, 50.3), turned to 135 degrees
- moved J8 128.6 mm to (210.3, 50.3), turned to 135 degrees
- moved U6 100.9 mm to (183.1, 60.0), turned to -90 degrees
- moved U15 97.9 mm to (189.2, 67.7), turned to 90 degrees
- moved D12 93.5 mm to (181.4, 69.8), turned to 90 degrees
- moved C15 85.8 mm to (189.2, 65.0)
- moved C14 85.5 mm to (189.2, 70.5)
- moved U4 84.6 mm to (178.4, 62.2), turned to -90 degrees
- moved U10 84.3 mm to (185.1, 67.7), turned to 90 degrees
- moved R43 84.2 mm to (176.9, 47.0), turned to -90 degrees
- moved R25 83.1 mm to (183.0, 70.0), turned to 90 degrees
- moved C19 79.0 mm to (180.9, 63.1), turned to -90 degrees
- moved C62 75.6 mm to (185.5, 64.9), turned to 180 degrees
- moved C63 75.4 mm to (185.5, 70.5), turned to 180 degrees
- moved U11 73.9 mm to (156.6, 55.5)
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Connections:
- R44 pad 5: SDMMC1_D2 -> SDMMC1_CMD
- R44 pad 6: SDMMC1_D3 -> SDMMC1_CLK
- R44 pad 7: SDMMC1_CLK -> SDMMC1_D3
- R44 pad 8: SDMMC1_CMD -> SDMMC1_D2
- SW3 pad 2: +3.3V -> +1V8
- SW4 pad 2: +3.3V -> +1V8
- SW6 pad 1: +3.3V -> +1V8
- SW7 pad 1: +3.3V -> +1V8
- U8 pad 20: unconnected-(U8-PA4-Pad20) -> RY_STICK
- U8 pad 21: unconnected-(U8-PA5-Pad21) -> RX_STICK
- U8 pad 22: unconnected-(U8-PA6-Pad22) -> LiPo_OBSERVE
- U8 pad 23: unconnected-(U8-PA7-Pad23) -> R1_BUTTON
- U8 pad 24: unconnected-(U8-PC4-Pad24) -> R2_BUTTON
- U8 pad 25: unconnected-(U8-PC5-Pad25) -> R3_BUTTON
- U8 pad 26: unconnected-(U8-PB0-Pad26) -> R4_BUTTON
- U8 pad 28: unconnected-(U8-PB2-Pad28) -> R_PUSH
- U8 pad 29: unconnected-(U8-PB10-Pad29) -> R_PUSH_HOME
- U8 pad 56: unconnected-(U8-PB4-Pad56) -> L8_BUTTON
- U8 pad 57: unconnected-(U8-PB5-Pad57) -> L7_BUTTON
- U8 pad 58: unconnected-(U8-PB6-Pad58) -> L6_BUTTON
- U8 pad 59: unconnected-(U8-PB7-Pad59) -> L5_BUTTON
- U8 pad 61: unconnected-(U8-PB8-Pad61) -> L_PUSH_HOME
- U8 pad 62: unconnected-(U8-PB9-Pad62) -> L_PUSH
- U8 pad 8: unconnected-(U8-PC0-Pad8) -> LY_STICK
- U8 pad 9: unconnected-(U8-PC1-Pad9) -> LX_STICK
Routing:
- net NRST: track 0.00 -> 137.0 mm, vias 0 -> 2
- net +5V: track 0.00 -> 106.0 mm, vias 0 -> 3
- net +1V8: track 4.34 -> 110.0 mm, vias 0 -> 7
- net SWCLK: track 0.00 -> 70.1 mm, vias 0 -> 1
- net R_PUSH: track 0.00 -> 67.1 mm, vias 0 -> 1
- net SWDIO: track 0.00 -> 65.8 mm, vias 0 -> 1
- net L_PUSH: track 0.00 -> 63.7 mm
- net BT_UART_CTS: track 0.00 -> 55.8 mm, vias 0 -> 2
- net BT_UART_RTS: track 0.00 -> 54.9 mm, vias 0 -> 2
- net BT_UART_RXD: track 0.00 -> 51.6 mm, vias 0 -> 2
- net BT_UART_TXD: track 0.00 -> 45.4 mm, vias 0 -> 2
- net Serial_TXD: track 0.00 -> 44.4 mm, vias 0 -> 2
- net Serial_RXD: track 0.00 -> 43.3 mm, vias 0 -> 2
- net Serial_RTS: track 0.00 -> 42.7 mm, vias 0 -> 2
- net R4_BUTTON: track 0.00 -> 40.1 mm, vias 0 -> 1
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- added copper zone on B.Cu, net GND
- added copper zone on F.Cu, net GND
- added copper zone on In1.Cu, net GND
- added copper zone on In2.Cu, net GND
