File: PCB/robo-con-Wi-Fi-v2/robo-con-Wi-Fi-v2.kicad_pcb (KiCad board)
At the start: 4 copper layers, 86 x 62 mm, 107 parts, among them J1 Conn_01x04, J11 Conn_01x05, J2 SMA-J, J3 Conn_01x05, J4 Conn_01x01, J5 Conn_01x02, J6 Conn_01x01, J8 Conn_01x01, J9 Conn_01x01, SW1 SW_Push, SW3 SW_Push, SW4 SW_Push, SW5 SW_Push_SPDT, SW6 SW_Push_SPDT, SW7 SW_Push_SPDT, U10 MCP73831-2-OT, U11 LM66100DCK, U15 LM66100DCK, U18 USB_Type-C, U2 LBEE5HY2FY, U3 FT234XD, U4 MCP1727-1802xMF, U5 RKJXV122400R, U6 LD39200PU33R, U7 RKJXV122400R, U8 STM32H7A3RGTx, Y2 XRCGB25M000FFS1AR0

Commit message: update PCB
Parts:
- removed D15: W, Diode_SMD:D_0603_1608Metric_Pad1.05x0.95mm_HandSolder
- removed D18: R, Diode_SMD:D_0603_1608Metric_Pad1.05x0.95mm_HandSolder
- removed R22, R36: 1k, Resistor_SMD:R_0402_1005Metric_Pad0.72x0.64mm_HandSolder
- D10, D13: value B -> O
- moved D11 103.1 mm to (183.2, 43.2), turned to -90 degrees
- moved R21 98.4 mm to (183.2, 46.8), turned to 90 degrees
- moved D16 86.7 mm to (181.2, 87.0), turned to -90 degrees
- moved D13 84.8 mm to (159.8, 44.4), turned to 90 degrees
- moved D10 82.4 mm to (161.9, 44.4), turned to 90 degrees
- moved R35 80.3 mm to (181.2, 83.6), turned to 90 degrees
- moved R11 78.9 mm to (161.9, 47.7), turned to -90 degrees
- moved R32 71.1 mm to (159.8, 47.7), turned to -90 degrees
- moved D5 68.7 mm to (143.0, 57.3), turned to 180 degrees
- moved D3 67.0 mm to (143.0, 55.1), turned to 180 degrees
- moved D1 65.5 mm to (143.0, 52.9), turned to 180 degrees
- moved D14 63.8 mm to (143.0, 59.4), turned to 180 degrees
- moved R6 59.6 mm to (146.4, 57.3)
- moved R4 58.6 mm to (146.4, 55.1)
- moved R2 57.6 mm to (146.4, 52.9)
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Connections:
- net LED3 renamed LEDWLTX
- net LED4 renamed LEDWLRX
- net LEDLiPo_GOOD renamed LEDLiPo
- U8 pad 2: unconnected-(U8-PC13-Pad2) -> LP_STICK
- U8 pad 27: unconnected-(U8-PB1-Pad27) -> RP_STICK
- U8 pad 36: unconnected-(U8-PB15-Pad36) -> BT_ON
- U8 pad 37: unconnected-(U8-PC6-Pad37) -> WL_ON
Routing:
- net RP_STICK: track 0.00 -> 46.7 mm, vias 0 -> 1
- net WL_ON: track 3.78 -> 43.7 mm, vias 1 -> 2
- net BT_ON: track 7.13 -> 46.5 mm, vias 0 -> 2
- net LP_STICK: track 0.00 -> 28.2 mm
- net LED0: track 0.00 -> 14.0 mm
- net LED1: track 0.00 -> 12.6 mm
- net LED2: track 0.00 -> 11.1 mm
- net LEDWL: track 0.00 -> 10.3 mm
- net LEDUSB: track 0.00 -> 8.77 mm
- net Net-(D11-A): track 0.00 -> 2.10 mm
- net Net-(D5-K): track 0.00 -> 2.01 mm
- net Net-(D3-K): track 0.00 -> 2.01 mm
- net Net-(D17-K): track 0.00 -> 2.01 mm
- net Net-(D14-K): track 0.00 -> 2.01 mm
- net Net-(D1-K): track 0.00 -> 2.01 mm
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
Commit message: up
Parts:
- added REF**: MountingHole_2.2mm_M2, MountingHole:MountingHole_2.2mm_M2, F.Cu at (133.0, 53.0)
- added REF**: MountingHole_2.2mm_M2, MountingHole:MountingHole_2.2mm_M2, F.Cu at (133.0, 87.0)
- added REF**: MountingHole_2.2mm_M2, MountingHole:MountingHole_2.2mm_M2, F.Cu at (207.0, 53.0)
- added REF**: MountingHole_2.2mm_M2, MountingHole:MountingHole_2.2mm_M2, F.Cu at (207.0, 87.0)
- moved G*** 121.2 mm to (199.3, 51.2)
- moved G*** 110.7 mm to (194.9, 61.4)
- moved R21 4.20 mm to (180.8, 50.2)
- moved D11 4.20 mm to (180.8, 46.6)
- moved D1 1.36 mm to (144.3, 52.7)
- moved D14 1.36 mm to (144.3, 59.2)
- moved D17 1.36 mm to (144.3, 61.4)
- moved D3 1.36 mm to (144.3, 54.9)
- moved D5 1.36 mm to (144.3, 57.0)
- moved R2 1.36 mm to (147.8, 52.7)
- moved R33 1.36 mm to (147.8, 59.2)
- moved R34 1.36 mm to (147.8, 61.4)
- moved R4 1.36 mm to (147.8, 54.9)
- moved R6 1.36 mm to (147.8, 57.0)
- moved J4 0.30 mm to (210.6, 50.2), turned to -45 degrees
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Connections:
- U8 pad 10: unconnected-(U8-PC2-Pad10) -> LEDWLRX
- U8 pad 11: unconnected-(U8-PC3-Pad11) -> LEDWLTX
- U8 pad 3: unconnected-(U8-PC14-Pad3) -> LEDWL
- U8 pad 33: unconnected-(U8-PB12-Pad33) -> LEDLiPo
- U8 pad 4: unconnected-(U8-PC15-Pad4) -> LED2
- U8 pad 40: unconnected-(U8-PA8-Pad40) -> LED0
- U8 pad 50: unconnected-(U8-PA15-Pad50) -> LED1
- U8 pad 55: unconnected-(U8-PB3-Pad55) -> LEDUSB
Routing:
- net +1V8: track 110.7 -> 357.6 mm, vias 7 -> 9
- net +3.3V: track 30.2 -> 163.9 mm, vias 0 -> 6
- net LEDWLTX: track 0.00 -> 39.2 mm, vias 0 -> 2
- net LEDWLRX: track 0.00 -> 39.1 mm, vias 0 -> 2
- net LEDLiPo: track 0.00 -> 26.3 mm, vias 0 -> 3
- net LED2: track 11.1 -> 34.2 mm, vias 0 -> 2
- net LEDWL: track 10.3 -> 32.4 mm, vias 0 -> 2
- net LED0: track 14.0 -> 31.3 mm
- net LEDUSB: track 8.77 -> 23.5 mm, vias 0 -> 2
- net LED1: track 12.6 -> 26.8 mm, vias 0 -> 2
- net +5V: track 106.3 -> 111.6 mm
- net NRST: track 137.0 -> 139.8 mm
- net unconnected-(U8-PB3-Pad55): track 1.97 -> 0.00 mm, vias 1 -> 0
- net unconnected-(U8-PA15-Pad50): track 1.95 -> 0.00 mm, vias 1 -> 0
- net Net-(D16-K): track 0.00 -> 1.87 mm
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Other:
- board text added: "+3.3V"
- board text added: "+BUS"
- board text added: "GND"
- board text added: "LED0"
- board text added: "LED1"
- board text added: "LED2"
- board text added: "LiPo"
- board text added: "NRST"
- board text added: "POWER"
- board text added: "RXWL"
- board text added: "Robo-Con-Wi-Fi6E"
- board text added: "SWCLK"
- board text added: "SWDIO"
- board text added: "TXWL"
- board text added: "USB"
- board text added: "Wi-Fi"
